File: SL_ADC_DE10Lite.kicad_pcb (KiCad board)
At the start: 4 copper layers, 98 x 67 mm, 26 parts, among them J1 DE10Lite header, J2 Analog header

Commit message: Board outline error?
Parts:
- removed R1: 10, Resistor_SMD:R_0508_1220Metric
- removed R2, R3: 10k, Resistor_SMD:R_0508_1220Metric
Routing:
- net /DGND: track 88.7 -> 63.3 mm, vias 4 -> 3
Other:
- board text removed: "10Ohm used to reduce noise for the DVDD pin"
- board text removed: "Pull down resistor for internal reference buffers in hardware mode?"
- board text removed: "Pull up resistor for internal reference buffers in hardware mode?"

Commit message: Generated step file
Other:
- outline, holes or cut-outs redrawn
- board text added: "A0 A0"
- board text added: "A1 A1"
- board text added: "AGND"
- board text added: "B0 B0"
- board text added: "B1 B1"
- board text added: "C0 C0"
- board text added: "DB0 DB1"
- board text added: "DB10 DB11"
- board text added: "DB12 DB13"
- board text added: "DB14 DB15"
- board text added: "DB2 DB3"
- board text added: "DB4 DB5"
- board text added: "DB6 DB7"
- board text added: "DB8 DB9"
- board text added: "DGND 5V"
- board text added: "DGND DVDD"
- board text added: "HVDD HVDD"
- board text added: "HVSS HVSS"
- board text added: "I2C1 I2C4"
- board text added: "I2C2 I2C3"
- board text added: "I2C4 I2C1"
- board text added: "I2C5 X"
- board text added: "IO20 X"
- board text added: "IO22 I2C5"
- board text added: "IO23 IO25"
- board text added: "IO24 IO19"
- board text added: "IO27 I226"
- board text added: "IO29 I228"
- board text added: "ZZZ IO21"
- board text added: "~{CS}/~{F5} ~{RD}"
