File: SL_ADC_DE10Lite.kicad_sch (KiCad schematic)
At the start: 24 parts, among them J1 DE10Lite header, J2 Conn_02x14_Odd_Even, J3 Conn_02x04_Odd_Even

Commit message: set HVDD to AVDD to share power supply and also updated PCB doc from schematic, re-routing and connecting AVDD to power needed still
Parts:
- removed J3: Conn_02x04_Odd_Even, Connector_PinHeader_2.54mm:PinHeader_2x04_P2.54mm_Horizontal, symbol Connector_Generic:Conn_02x04_Odd_Even
Connections:
- net HVDD is gone; now on net AVDD: C18.1, C20.1, IC1.48 (HVDD), J2.25 (Pin_25), J2.27 (Pin_27)
Other:
- note added: "The chip will be powered by 5V coming from the HVDD pin which will also be the maximum of its measurable range"
Changed lines of the file:
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@@
 		)
 	)
+	(text "The chip will be powered\nby 5V coming from the HVDD pin which will\nalso be the maximum of its measurable range\n"
+		(exclude_from_sim no)
+		(at 99.822 168.402 0)
+		(effects
+			(font
+				(size 0.762 0.762)
+			)
+		)
+	)
 	(text "ADC\n"
 		(exclude_from_sim no)
@@
 	(wire
 		(pts
+			(xy 91.44 162.56) (xy 100.33 162.56)
+		)
+		(stroke
+			(width 0)
+			(type default)
+		)
+	)
+	(wire
+		(pts
 			(xy 241.3 41.91) (xy 241.3 48.26)
 		)
@@
 		)
 	)
-	(label "CH_D1"
-		(at 87.63 130.81 180)
-		(effects
-			(font
-				(size 1.27 1.27)
-			)
-			(justify right bottom)
-		)
-	)
 	(label "HVDD"
 		(at 116.84 41.91 0)
@@
 		)
 	)
-	(label "CH_B1"
-		(at 100.33 138.43 0)
-		(effects
-			(font
-				(size 1.27 1.27)
-			)
-			(justify left bottom)
-		)
-	)
 	(label "~{RD}"
 		(at 44.45 135.89 180)
@@
 		)
 	)
-	(label "CH_D0"
-		(at 87.63 133.35 180)
-		(effects
-			(font
-				(size 1.27 1.27)
-			)
-			(justify right bottom)
-		)
-	)
 	(label "DVDD"
 		(at 116.84 130.81 180)
@@
 		)
 	)
+	(label "AVDD"
+		(at 100.33 162.56 0)
+		(effects
+			(font
+				(size 1.27 1.27)
+			)
+			(justify left bottom)
+		)
+	)
 	(label "I2C1"
 		(at 44.45 179.07 180)
@@
 		)
 	)
-	(label "CH_C1"
-		(at 87.63 135.89 180)
-		(effects
-			(font
-				(size 1.27 1.27)
-			)
-			(justify right bottom)
-		)
-	)
 	(label "AGND"
 		(at 184.15 54.61 0)
@@
 		)
 	)
+	(label "HVDD"
+		(at 91.44 162.56 0)
+		(effects
+			(font
+				(size 1.27 1.27)
+			)
+			(justify left bottom)
+		)
+	)
 	(label "AGND"
 		(at 241.3 48.26 0)
@@
 		)
 	)
-	(label "CH_A1"
-		(at 100.33 133.35 0)
-		(effects
-			(font
-				(size 1.27 1.27)
-			)
-			(justify left bottom)
-		)
-	)
 	(label "CH_B1"
 		(at 129.54 153.67 0)
@@
 		)
 	)
-	(label "CH_A0"
-		(at 100.33 130.81 0)
-		(effects
-			(font
-				(size 1.27 1.27)
-			)
-			(justify left bottom)
-		)
-	)
 	(label "AGND"
 		(at 116.84 153.67 180)
@@
 		)
 	)
-	(label "CH_B0"
-		(at 100.33 135.89 0)
-		(effects
-			(font
-				(size 1.27 1.27)
-			)
-			(justify left bottom)
-		)
-	)
 	(label "HVSS"
 		(at 116.84 158.75 180)
@@
 		)
 	)
-	(label "CH_C0"
-		(at 87.63 138.43 180)
-		(effects
-			(font
-				(size 1.27 1.27)
-			)
-			(justify right bottom)
-		)
-	)
 	(label "AGND"
 		(at 116.84 52.07 0)
@@
 					(unit 1)
 				)
-			)
-		)
-	)
-	(symbol
-		(lib_id "Connector_Generic:Conn_02x04_Odd_Even")
-		(at 92.71 133.35 0)
-		(unit 1)
-		(body_style 1)
-		(exclude_from_sim no)
-		(in_bom yes)
-		(on_board yes)
-		(in_pos_files yes)
-		(dnp no)
-		(fields_autoplaced yes)
-		(property "Reference" "J3"
-			(at 93.98 124.46 0)
-			(show_name no)
-			(do_not_autoplace no)
-			(effects
-				(font
-					(size 1.27 1.27)
-				)
-			)
-		)
-		(property "Value" "Conn_02x04_Odd_Even"
-			(at 93.98 127 0)
-			(show_name no)
-			(do_not_autoplace no)
-			(effects
-				(font
-					(size 1.27 1.27)
-				)
-			)
-		)
-		(property "Footprint" "Connector_PinHeader_2.54mm:PinHeader_2x04_P2.54mm_Horizontal"
-			(at 92.71 133.35 0)
-			(hide yes)
-			(show_name no)
-			(do_not_autoplace no)
-			(effects
-				(font
-					(size 1.27 1.27)
-				)
-			)
-		)
-		(property "Datasheet" ""
-			(at 92.71 133.35 0)
-			(hide yes)
-			(show_name no)
-			(do_not_autoplace no)
-			(effects
-				(font
-					(size 1.27 1.27)
-				)
-			)
-		)
-		(property "Description" "Generic connector, double row, 02x04, odd/even pin numbering scheme (row 1 odd numbers, row 2 even numbers), script generated (kicad-library-utils/schlib/autogen/connector/)"
-			(at 92.71 133.35 0)
-			(hide yes)
-			(show_name no)
-			(do_not_autoplace no)
-			(effects
-				(font
-					(size 1.27 1.27)
-				)
-			)
-		)
-		(pin "5"
-		)
-		(pin "2"
-		)
-		(pin "4"
-		)
-		(pin "8"
-		)
-		(pin "6"
-		)
-		(pin "3"
-		)
-		(pin "1"
-		)
-		(pin "7"
-		)
-		(instances
-			(project "SL_ADC_DE10Lite"
-				(path "/9fa1cf44-a1cc-46e9-aa9b-d59a1c14c45e"
-					(reference "J3")
-					(unit 1)
-				)

Commit message: updated PCB to match foodtprint header pinout, flagged issues with ground planes only being on one layer and not being under all the relevant pins. Re-routing and ground plane re-shaping needed
Changed lines of the file:
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@@
+		)
+	)
+	(label "AVDD"
+		(at 116.84 163.83 180)
+		(effects
+			(font
+				(size 1.27 1.27)
+			)
+			(justify right bottom)
 		)
 	)
@@
 		(effects
 			(font
-				(size 1.27 1.27)
-			)
-			(justify right bottom)
-		)
-	)
-	(label "HVDD"
-		(at 116.84 163.83 180)
-		(effects
-			(font

Commit message: fixed some DRC issues
Connections:
- net DGND is gone; now on net AGND: C5.2, IC1.24 (DGND), J1.12 (Pin_12), J1.30 (Pin_30)
Other:
- note added: "AGND and DGND are joined at the bottom of the ADS8528"
Changed lines of the file:
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@@
+		)
+	)
+	(text "AGND and DGND are joined at the\nbottom of the ADS8528\n"
+		(exclude_from_sim no)
+		(at 98.044 155.956 0)
+		(effects
+			(font
+				(size 0.762 0.762)
+			)
 		)
 	)
@@
 	(wire
 		(pts
-			(xy 241.3 63.5) (xy 241.3 69.85)
+			(xy 91.44 151.13) (xy 100.33 151.13)
 		)
 		(stroke
@@
 		)
 	)
+	(wire
+		(pts
+			(xy 241.3 63.5) (xy 241.3 69.85)
+		)
+		(stroke
+			(width 0)
+			(type default)
+		)
+	)
 	(label "DB12"
 		(at 66.04 85.09 270)
@@
 		)
 	)
+	(label "DGND"
+		(at 100.33 151.13 0)
+		(effects
+			(font
+				(size 1.27 1.27)
+			)
+			(justify left bottom)
+		)
+	)
 	(label "CH_A0"
 		(at 116.84 57.15 0)
@@
 		)
 	)
+	(label "AGND"
+		(at 91.44 151.13 0)
+		(effects
+			(font
+				(size 1.27 1.27)
+			)
+			(justify left bottom)
+		)
+	)

Commit message: added 0 ohm jumper for REFN and increase via to ADC spacing while decrasing cap to ADC spacing
Parts:
- added R1: 0, LED_SMD:LED_0805_2012Metric, symbol Device:R
Connections:
- net AGND: now also R1.2
- net REFN: now also R1.1
Other:
- note added: "Unsure if REFN needs to be connected or not putting a 0 ohm resistor to make it configurable"
Changed lines of the file:
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@@
 		)
 	)
+	(text "Unsure if REFN needs to \nbe connected or not\nputting a 0 ohm resistor to\nmake it configurable"
+		(exclude_from_sim no)
+		(at 252.984 89.408 0)
+		(effects
+			(font
+				(size 1.27 1.27)
+			)
+			(justify left)
+		)
+	)
 	(text "(pin 63)"
 		(exclude_from_sim no)
@@
 	(wire
 		(pts
+			(xy 241.3 85.09) (xy 241.3 87.63)
+		)
+		(stroke
+			(width 0)
+			(type default)
+		)
+	)
+	(wire
+		(pts
 			(xy 261.62 63.5) (xy 261.62 69.85)
 		)
@@
 	(wire
 		(pts
+			(xy 241.3 97.79) (xy 241.3 95.25)
+		)
+		(stroke
+			(width 0)
+			(type default)
+		)
+	)
+	(wire
+		(pts
 			(xy 241.3 63.5) (xy 241.3 69.85)
 		)
@@
 		)
 	)
+	(label "AGND"
+		(at 241.3 97.79 0)
+		(effects
+			(font
+				(size 1.27 1.27)
+			)
+			(justify left bottom)
+		)
+	)
 	(label "GPIO(20)-BUSY{slash}INT"
 		(at 57.15 161.29 0)
@@
 					(unit 1)
 				)
+			)
+		)
+	)
+	(symbol
+		(lib_id "Device:R")
+		(at 241.3 91.44 0)
+		(unit 1)
+		(body_style 1)
+		(exclude_from_sim no)
+		(in_bom yes)
+		(on_board yes)
+		(in_pos_files yes)
+		(dnp no)
+		(fields_autoplaced yes)
+		(property "Reference" "R1"
+			(at 243.84 90.1699 0)
+			(show_name no)
+			(do_not_autoplace no)
+			(effects
+				(font
+					(size 1.27 1.27)
+				)
+				(justify left)
+			)
+		)
+		(property "Value" "0"
+			(at 243.84 92.7099 0)
+			(show_name no)
+			(do_not_autoplace no)
+			(effects
+				(font
+					(size 1.27 1.27)
+				)
+				(justify left)
+			)
+		)
+		(property "Footprint" "LED_SMD:LED_0805_2012Metric"
+			(at 239.522 91.44 90)
+			(hide yes)
+			(show_name no)
+			(do_not_autoplace no)
+			(effects
+				(font
+					(size 1.27 1.27)
+				)
+			)
+		)
+		(property "Datasheet" ""
+			(at 241.3 91.44 0)
+			(hide yes)
+			(show_name no)
+			(do_not_autoplace no)
+			(effects
+				(font
+					(size 1.27 1.27)
+				)
+			)
+		)
+		(property "Description" "Resistor"
+			(at 241.3 91.44 0)
+			(hide yes)
+			(show_name no)
+			(do_not_autoplace no)
+			(effects
+				(font
+					(size 1.27 1.27)
+				)
+			)
+		)
+		(pin "1"
+		)
+		(pin "2"
+		)
+		(instances
+			(project "SL_ADC_DE10Lite"
+				(path "/9fa1cf44-a1cc-46e9-aa9b-d59a1c14c45e"
+					(reference "R1")
+					(unit 1)
+				)
