File: _autosave-SL_ADC_DE10Lite.kicad_pcb (KiCad board)
At the start: 4 copper layers, 98 x 67 mm, 34 parts, among them J1 DE10Lite header, J2 Conn_02x14_Odd_Even

Commit message: added 0 ohm jumper for REFN and increase via to ADC spacing while decrasing cap to ADC spacing
Parts:
- moved ? 2.24 mm to (125.2, 89.3)
Changed lines of the file:
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@@
 	(footprint "PCBDrawings:SubbotsFish"
 		(layer "F.Cu")
-		(at 125 91.5)
+		(at 125.248733 89.275896)
 		(property "Reference" ""
 			(at 0 0 0)
@@
 			(at -3.5 -2 0)
 			(layer "F.SilkS")
-			(effects
-				(font
+			(hide yes)
+			(effects
+				(font

Commit message: fixed DGND DVDD and 5V pin placements to match DE10 in real life
Parts:
- moved ? 2.24 mm to (125.0, 91.5)
Connections:
- J1 pad 11: /DE10_5V -> /AGND
- J1 pad 12: /AGND -> /DVDD
- J1 pad 29: /DVDD -> unconnected-(J1-Pin_29-Pad29)
- J1 pad 30: /AGND -> /DE10_5V
Routing:
- net (no net): track 0.00 -> 31.0 mm
- net /DVDD: track 101.4 -> 119.0 mm

Commit message: fixed header issue
Parts:
- J1: footprint Connector_PinSocket_2.54mm:PinSocket_2x20_P2.54mm_Vertical -> Connector_PinHeader_2.54mm:PinHeader_2x20_P2.54mm_Vertical; moved to F.Cu
- moved J1 48.3 mm to (84.5, 55.0)
Connections:
- J1 pad 1: /GPIO(19)-~{PAR}/SER -> /I2C4
- J1 pad 10: /DB12 -> /GPIO(26)-CONVSTA
- J1 pad 11: /AGND -> /DE10_5V
- J1 pad 12: /DVDD -> /AGND
- J1 pad 13: /DB11 -> /ASLEEP
- J1 pad 14: /DB10 -> /GPIO(21)-RANGE/XCLK
- J1 pad 15: /DB9 -> /GPIO(20)-BUSY/INT
- J1 pad 16: /DB8 -> unconnected-(J1-Pin_16-Pad16)
- J1 pad 17: /DB7 -> /DB0
- J1 pad 18: /DB6 -> /DB1
- J1 pad 19: /DB5 -> /DB2
- J1 pad 2: /GPIO(24)-~{STBY} -> /I2C1
- J1 pad 20: /DB4 -> /DB3
- J1 pad 21: /DB3 -> /DB4
- J1 pad 22: /DB2 -> /DB5
- J1 pad 23: /DB1 -> /DB6
- J1 pad 24: /DB0 -> /DB7
- J1 pad 25: unconnected-(J1-Pin_25-Pad25) -> /DB8
- J1 pad 26: /GPIO(20)-BUSY/INT -> /DB9
- J1 pad 27: /GPIO(21)-RANGE/XCLK -> /DB10
- J1 pad 28: /ASLEEP -> /DB11
- J1 pad 29: unconnected-(J1-Pin_29-Pad29) -> /DVDD
- J1 pad 3: /GPIO(25)-RESET -> /I2C2
- J1 pad 30: /DE10_5V -> /AGND
- J1 pad 31: /GPIO(26)-CONVSTA -> /DB12
- J1 pad 32: /GPIO(27)-CONVSTB -> /DB13
- J1 pad 33: /GPIO(28)-CONVSTC -> /DB14
- J1 pad 34: /GPIO(29)-CONVSTD -> /DB15
- J1 pad 35: /I2C5 -> /~{CS}/~{F5}
- J1 pad 36: /GPIO(22)-~{HW}/SW -> /~{RD}
- J1 pad 37: /I2C3 -> /GPIO(23)-REFEN/~{WR}
- J1 pad 38: /I2C2 -> /GPIO(25)-RESET
- J1 pad 39: /I2C1 -> /GPIO(24)-~{STBY}
- J1 pad 4: /GPIO(23)-REFEN/~{WR} -> /I2C3
- J1 pad 40: /I2C4 -> /GPIO(19)-~{PAR}/SER
- J1 pad 5: /~{RD} -> /GPIO(22)-~{HW}/SW
- J1 pad 6: /~{CS}/~{F5} -> /I2C5
- J1 pad 7: /DB15 -> /GPIO(29)-CONVSTD
- J1 pad 8: /DB14 -> /GPIO(28)-CONVSTC
- J1 pad 9: /DB13 -> /GPIO(27)-CONVSTB
Routing:
- net (no net): track 31.0 -> 0.00 mm
